Commit message: Use primitive forearm visuals and extended gripper bodies

File: isaac_lab_data_collection/src/my_robot_description/urdf/biped_s40_primitives.urdf (robot description, URDF)
Before this commit: robot my_robot_description, 50 links, 49 joints
Links:
- link base_link: geometry visual box size=0.25 0.18 0.4
- link camera: geometry visual box size=0.06 0.04 0.04
- link leg_l1_link: geometry visual cylinder length=0.12 radius=0.05
- link leg_l2_link: geometry visual box size=0.12 0.08 0.18
- link leg_l3_link: geometry visual cylinder length=0.24 radius=0.045
- link leg_l4_link: geometry visual box size=0.1 0.08 0.2
- link leg_l5_link: geometry visual box size=0.09 0.07 0.12
- link leg_l6_link: geometry visual box size=0.16 0.09 0.05
- link leg_r1_link: geometry visual cylinder length=0.12 radius=0.05
- link leg_r2_link: geometry visual box size=0.12 0.08 0.18
- link leg_r3_link: geometry visual cylinder length=0.24 radius=0.045
- link leg_r4_link: geometry visual box size=0.1 0.08 0.2
- link leg_r5_link: geometry visual box size=0.09 0.07 0.12
- link leg_r6_link: geometry visual box size=0.16 0.09 0.05
- link zarm_l1_link: geometry visual cylinder length=0.12 radius=0.04
- link zarm_l2_link: geometry visual box size=0.1 0.08 0.14
- link zarm_l3_link: geometry visual cylinder length=0.26 radius=0.04
- link zarm_l4_link: geometry visual box size=0.08 0.08 0.18
- link zarm_l5_link: geometry visual box size=0.06 0.08 0.16
- link zarm_l6_link: geometry visual cylinder length=0.14 radius=0.03
- link zarm_l7_end_effector: geometry collision box size=0.04 0.06 0.04; visual box size=0.04 0.06 0.04
- link zarm_l7_link: geometry visual box size=0.05 0.07 0.14
- link zarm_r1_link: geometry visual cylinder length=0.12 radius=0.04
- link zarm_r2_link: geometry visual box size=0.1 0.08 0.14
- link zarm_r3_link: geometry visual cylinder length=0.26 radius=0.04
- link zarm_r4_link: geometry visual box size=0.08 0.08 0.18
- link zarm_r5_link: geometry visual box size=0.06 0.08 0.16
- link zarm_r6_link: geometry visual cylinder length=0.14 radius=0.03
- link zarm_r7_end_effector: geometry collision box size=0.04 0.06 0.04; visual box size=0.04 0.06 0.04
- link zarm_r7_link: geometry visual box size=0.05 0.07 0.14
- link zhead_1_link: geometry visual cylinder length=0.1 radius=0.05
- link zhead_2_link: geometry visual box size=0.16 0.14 0.2
