Commit message: upd model

File: isaac_lab_data_collection/install/my_robot_description/share/my_robot_description/urdf/biped_s40.urdf (robot description, URDF)
Before this commit: robot biped_s40, 46 links, 45 joints
Links:
- link base_link: geometry visual cylinder length=0.15 radius=0.03; visual sphere radius=0.03
- link camera: geometry visual cylinder length=0.15 radius=0.03; visual sphere radius=0.03
- link camera_base: geometry collision cylinder length=0.15 radius=0.03; visual cylinder length=0.15 radius=0.03
- link leg_l1_link: geometry visual cylinder length=0.15 radius=0.03; visual sphere radius=0.03
- link leg_l2_link: geometry visual cylinder length=0.15 radius=0.03; visual sphere radius=0.03
- link leg_l3_link: geometry visual cylinder length=0.15 radius=0.03; visual sphere radius=0.03
- link leg_l4_link: geometry visual cylinder length=0.15 radius=0.03; visual sphere radius=0.03
- link leg_l5_link: geometry visual cylinder length=0.15 radius=0.03; visual sphere radius=0.03
- link leg_l6_link: geometry visual cylinder length=0.15 radius=0.03; visual sphere radius=0.03
- link leg_r1_link: geometry visual cylinder length=0.15 radius=0.03; visual sphere radius=0.03
- link leg_r2_link: geometry visual cylinder length=0.15 radius=0.03; visual sphere radius=0.03
- link leg_r3_link: geometry visual cylinder length=0.15 radius=0.03; visual sphere radius=0.03
- link leg_r4_link: geometry visual cylinder length=0.15 radius=0.03; visual sphere radius=0.03
- link leg_r5_link: geometry visual cylinder length=0.15 radius=0.03; visual sphere radius=0.03
- link leg_r6_link: geometry visual cylinder length=0.15 radius=0.03; visual sphere radius=0.03
- link zarm_l1_link: geometry visual cylinder length=0.15 radius=0.03; visual sphere radius=0.03
- link zarm_l2_link: geometry visual cylinder length=0.15 radius=0.03; visual sphere radius=0.03
- link zarm_l3_link: geometry visual cylinder length=0.15 radius=0.03; visual sphere radius=0.03
- link zarm_l4_link: geometry visual cylinder length=0.15 radius=0.03; visual sphere radius=0.03
- link zarm_l5_link: geometry visual cylinder length=0.15 radius=0.03; visual sphere radius=0.03
- link zarm_l6_link: geometry visual cylinder length=0.15 radius=0.03; visual sphere radius=0.03
- link zarm_l7_link: geometry visual cylinder length=0.15 radius=0.03; visual sphere radius=0.03
- link zarm_r1_link: geometry visual cylinder length=0.15 radius=0.03; visual sphere radius=0.03
- link zarm_r2_link: geometry visual cylinder length=0.15 radius=0.03; visual sphere radius=0.03
- link zarm_r3_link: geometry visual cylinder length=0.15 radius=0.03; visual sphere radius=0.03
- link zarm_r4_link: geometry visual cylinder length=0.15 radius=0.03; visual sphere radius=0.03
- link zarm_r5_link: geometry visual cylinder length=0.15 radius=0.03; visual sphere radius=0.03
- link zarm_r6_link: geometry visual cylinder length=0.15 radius=0.03; visual sphere radius=0.03
- link zarm_r7_link: geometry visual cylinder length=0.15 radius=0.03; visual sphere radius=0.03
- link zhead_1_link: geometry visual cylinder length=0.15 radius=0.03; visual sphere radius=0.03
- link zhead_2_link: geometry visual cylinder length=0.15 radius=0.03; visual sphere radius=0.03

Commit message: old model with meshes

File: isaac_lab_data_collection/install/my_robot_description/share/my_robot_description/urdf/biped_s40.urdf (robot description, URDF)
Before this commit: robot my_robot_description, 46 links, 45 joints
Links:
- link base_link: geometry visual mesh filename=package://my_robot_description/meshes/base_link.STL
- link camera: geometry visual mesh filename=package://my_robot_description/meshes/camera.STL
- link camera_base: geometry collision mesh filename=package://my_robot_description/meshes/camera_base.STL; visual mesh filename=package://my_robot_description/meshes/camera_base.STL
- link leg_l1_link: geometry visual mesh filename=package://my_robot_description/meshes//l_leg_roll.STL
- link leg_l2_link: geometry visual mesh filename=package://my_robot_description/meshes/l_leg_yaw.STL
- link leg_l3_link: geometry visual mesh filename=package://my_robot_description/meshes/l_leg_pitch.STL
- link leg_l4_link: geometry visual mesh filename=package://my_robot_description/meshes/l_knee.STL
- link leg_l5_link: geometry visual mesh filename=package://my_robot_description/meshes/l_foot_pitch.STL
- link leg_l6_link: geometry visual mesh filename=package://my_robot_description/meshes/l_foot_roll.STL
- link leg_r1_link: geometry visual mesh filename=package://my_robot_description/meshes/r_leg_roll.STL
- link leg_r2_link: geometry visual mesh filename=package://my_robot_description/meshes/r_leg_yaw.STL
- link leg_r3_link: geometry visual mesh filename=package://my_robot_description/meshes/r_leg_pitch.STL
- link leg_r4_link: geometry visual mesh filename=package://my_robot_description/meshes/r_knee.STL
- link leg_r5_link: geometry visual mesh filename=package://my_robot_description/meshes/r_foot_pitch.STL
- link leg_r6_link: geometry visual mesh filename=package://my_robot_description/meshes/r_foot_roll.STL
- link zarm_l1_link: geometry visual mesh filename=package://my_robot_description/meshes/l_arm_pitch.STL
- link zarm_l2_link: geometry visual mesh filename=package://my_robot_description/meshes/l_arm_roll.STL
- link zarm_l3_link: geometry visual mesh filename=package://my_robot_description/meshes/l_arm_yaw.STL
- link zarm_l4_link: geometry visual mesh filename=package://my_robot_description/meshes/l_forearm.STL
- link zarm_l5_link: geometry visual mesh filename=package://my_robot_description/meshes/l_hand_yaw.STL
- link zarm_l6_link: geometry visual mesh filename=package://my_robot_description/meshes/l_hand_pitch.STL
- link zarm_l7_link: geometry visual mesh filename=package://my_robot_description/meshes/l_hand_roll.STL
- link zarm_r1_link: geometry visual mesh filename=package://my_robot_description/meshes/r_arm_pitch.STL
- link zarm_r2_link: geometry visual mesh filename=package://my_robot_description/meshes/r_arm_roll.STL
- link zarm_r3_link: geometry visual mesh filename=package://my_robot_description/meshes/r_arm_yaw.STL
- link zarm_r4_link: geometry visual mesh filename=package://my_robot_description/meshes/r_forearm.STL
- link zarm_r5_link: geometry visual mesh filename=package://my_robot_description/meshes/r_hand_yaw.STL
- link zarm_r6_link: geometry visual mesh filename=package://my_robot_description/meshes/r_hand_pitch.STL
- link zarm_r7_link: geometry visual mesh filename=package://my_robot_description/meshes/r_hand_roll.STL
- link zhead_1_link: geometry visual mesh filename=package://my_robot_description/meshes/head_yaw.STL
- link zhead_2_link: geometry visual mesh filename=package://my_robot_description/meshes/head_pitch.STL

File: simulation_data_collection/src/biped_s40/urdf/biped_s40.urdf (robot description, URDF)
Before this commit: robot biped_s40, 46 links, 45 joints
Links:
- link base_link: geometry visual mesh filename=package://kuavo_assets/models/biped_s40/meshes/base_link.STL
- link camera: geometry visual mesh filename=package://kuavo_assets/models/biped_s40/meshes/camera.STL
- link camera_base: geometry collision mesh filename=package://kuavo_assets/models/biped_s40/meshes/camera_base.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; visual mesh filename=package://kuavo_assets/models/biped_s40/meshes/camera_base.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
- link leg_l1_link: geometry visual mesh filename=package://kuavo_assets/models/biped_s40/meshes/l_leg_roll.S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
- link leg_l2_link: geometry visual mesh filename=package://kuavo_assets/models/biped_s40/meshes/l_leg_yaw.STL
- link leg_l3_link: geometry visual mesh filename=package://kuavo_assets/models/biped_s40/meshes/l_leg_pitch.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
- link leg_l4_link: geometry visual mesh filename=package://kuavo_assets/models/biped_s40/meshes/l_knee.STL
- link leg_l5_link: geometry visual mesh filename=package://kuavo_assets/models/biped_s40/meshes/l_foot_pitch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
- link leg_l6_link: geometry visual mesh filename=package://kuavo_assets/models/biped_s40/meshes/l_foot_roll.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
- link leg_r1_link: geometry visual mesh filename=package://kuavo_assets/models/biped_s40/meshes/r_leg_roll.S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
- link leg_r2_link: geometry visual mesh filename=package://kuavo_assets/models/biped_s40/meshes/r_leg_yaw.STL
- link leg_r3_link: geometry visual mesh filename=package://kuavo_assets/models/biped_s40/meshes/r_leg_pitch.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
- link leg_r4_link: geometry visual mesh filename=package://kuavo_assets/models/biped_s40/meshes/r_knee.STL
- link leg_r5_link: geometry visual mesh filename=package://kuavo_assets/models/biped_s40/meshes/r_foot_pitch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
- link leg_r6_link: geometry visual mesh filename=package://kuavo_assets/models/biped_s40/meshes/r_foot_roll.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
- link zarm_l1_link: geometry visual mesh filename=package://kuavo_assets/models/biped_s40/meshes/l_arm_pitch.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
- link zarm_l2_link: geometry visual mesh filename=package://kuavo_assets/models/biped_s40/meshes/l_arm_roll.S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
- link zarm_l3_link: geometry visual mesh filename=package://kuavo_assets/models/biped_s40/meshes/l_arm_yaw.STL
- link zarm_l4_link: geometry visual mesh filename=package://kuavo_assets/models/biped_s40/meshes/l_forearm.STL
- link zarm_l5_link: geometry visual mesh filename=package://kuavo_assets/models/biped_s40/meshes/l_hand_yaw.S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
- link zarm_l6_link: geometry visual mesh filename=package://kuavo_assets/models/biped_s40/meshes/l_hand_pitch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
- link zarm_l7_link: geometry visual mesh filename=package://kuavo_assets/models/biped_s40/meshes/l_hand_roll.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
- link zarm_r1_link: geometry visual mesh filename=package://kuavo_assets/models/biped_s40/meshes/r_arm_pitch.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
- link zarm_r2_link: geometry visual mesh filename=package://kuavo_assets/models/biped_s40/meshes/r_arm_roll.S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
- link zarm_r3_link: geometry visual mesh filename=package://kuavo_assets/models/biped_s40/meshes/r_arm_yaw.STL
- link zarm_r4_link: geometry visual mesh filename=package://kuavo_assets/models/biped_s40/meshes/r_forearm.STL
- link zarm_r5_link: geometry visual mesh filename=package://kuavo_assets/models/biped_s40/meshes/r_hand_yaw.S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
- link zarm_r6_link: geometry visual mesh filename=package://kuavo_assets/models/biped_s40/meshes/r_hand_pitch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
- link zarm_r7_link: geometry visual mesh filename=package://kuavo_assets/models/biped_s40/meshes/r_hand_roll.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
- link zhead_1_link: geometry visual mesh filename=package://kuavo_assets/models/biped_s40/meshes/head_yaw.STL
- link zhead_2_link: geometry visual mesh filename=package://kuavo_assets/models/biped_s40/meshes/head_pitch.S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

Commit message: upd end effector

File: isaac_lab_data_collection/install/my_robot_description/share/my_robot_description/urdf/biped_s40.urdf (robot description, URDF)
Before this commit: robot biped_s40, 46 links, 45 joints
Links:
- added link zarm_l_finger_left, mass 0.05; collision box size=0.12 0.035 0.035; visual box size=0.07 0.03 0.03
- added link zarm_l_finger_right, mass 0.05; collision box size=0.12 0.035 0.035; visual box size=0.07 0.03 0.03
- added link zarm_r_finger_left, mass 0.05; collision box size=0.12 0.035 0.035; visual box size=0.07 0.03 0.03
- added link zarm_r_finger_right, mass 0.05; collision box size=0.12 0.035 0.035; visual box size=0.07 0.03 0.03
- link base_link: geometry visual mesh filename=package://my_robot_description/meshes/base_link.STL scale=1 1 1
- link camera: geometry visual mesh filename=package://my_robot_description/meshes/camera.STL scale=1 1 1
- link camera_base: geometry collision cylinder length=0.15 radius=0.03; visual mesh filename=package://my_robot_description/meshes/camera_base.STL scale=1 1 1
- link leg_l1_link: geometry visual mesh filename=package://my_robot_description/meshes/l_leg_roll.STL scale=1 1 1
- link leg_l2_link: geometry visual mesh filename=package://my_robot_description/meshes/l_leg_yaw.STL scale=1 1 1
- link leg_l3_link: geometry visual mesh filename=package://my_robot_description/meshes/l_leg_pitch.STL scale=1 1 1
- link leg_l4_link: geometry visual mesh filename=package://my_robot_description/meshes/l_knee.STL scale=1 1 1
- link leg_l5_link: geometry visual mesh filename=package://my_robot_description/meshes/l_foot_pitch.STL scale=1 1 1
- link leg_l6_link: geometry visual mesh filename=package://my_robot_description/meshes/l_foot_roll.STL scale=1 1 1
- link leg_r1_link: geometry visual mesh filename=package://my_robot_description/meshes/r_leg_roll.STL scale=1 1 1
- link leg_r2_link: geometry visual mesh filename=package://my_robot_description/meshes/r_leg_yaw.STL scale=1 1 1
- link leg_r3_link: geometry visual mesh filename=package://my_robot_description/meshes/r_leg_pitch.STL scale=1 1 1
- link leg_r4_link: geometry visual mesh filename=package://my_robot_description/meshes/r_knee.STL scale=1 1 1
- link leg_r5_link: geometry visual mesh filename=package://my_robot_description/meshes/r_foot_pitch.STL scale=1 1 1
- link leg_r6_link: geometry visual mesh filename=package://my_robot_description/meshes/r_foot_roll.STL scale=1 1 1
- link zarm_l1_link: geometry visual mesh filename=package://my_robot_description/meshes/l_arm_pitch.STL scale=1 1 1
- link zarm_l2_link: geometry visual mesh filename=package://my_robot_description/meshes/l_arm_roll.STL scale=1 1 1
- link zarm_l3_link: geometry visual mesh filename=package://my_robot_description/meshes/l_arm_yaw.STL scale=1 1 1
- link zarm_l4_link: geometry visual mesh filename=package://my_robot_description/meshes/l_forearm.STL scale=1 1 1
- link zarm_l5_link: geometry visual mesh filename=package://my_robot_description/meshes/l_hand_pitch.STL scale=1 1 1
- link zarm_l6_link: geometry collision box size=0.04 0.04 0.12; visual box size=0.04 0.04 0.12
- link zarm_l7_end_effector: mass None -> 0.2; geometry collision cylinder length=0.015 radius=0.02; visual cylinder length=0.015 radius=0.02
- link zarm_l7_link: geometry 
- link zarm_r1_link: geometry visual mesh filename=package://my_robot_description/meshes/r_arm_pitch.STL scale=1 1 1
- link zarm_r2_link: geometry visual mesh filename=package://my_robot_description/meshes/r_arm_roll.STL scale=1 1 1
- link zarm_r3_link: geometry visual mesh filename=package://my_robot_description/meshes/r_arm_yaw.STL scale=1 1 1
- link zarm_r4_link: geometry visual mesh filename=package://my_robot_description/meshes/r_forearm.STL scale=1 1 1
- link zarm_r5_link: geometry visual mesh filename=package://my_robot_description/meshes/r_hand_pitch.STL scale=1 1 1
- link zarm_r6_link: geometry collision box size=0.04 0.04 0.12; visual box size=0.04 0.04 0.12
- link zarm_r7_end_effector: mass None -> 0.2; geometry collision cylinder length=0.015 radius=0.02; visual cylinder length=0.015 radius=0.02
- link zarm_r7_link: geometry 
- link zhead_1_link: geometry visual mesh filename=package://my_robot_description/meshes/head_yaw.STL scale=1 1 1
- link zhead_2_link: geometry visual mesh filename=package://my_robot_description/meshes/head_pitch.STL scale=1 1 1
Joints:
- added joint zarm_l_finger_left_joint: type revolute, parent zarm_l7_end_effector, child zarm_l_finger_left, origin xyz=-0.02 0.035 0 rpy=0 0 0, axis 0 0 1, limit lower=0.0 upper=0.78539816339 effort=5.0 velocity=1.0
- added joint zarm_l_finger_right_joint: type revolute, parent zarm_l7_end_effector, child zarm_l_finger_right, origin xyz=-0.02 -0.035 0 rpy=0 0 0, axis 0 0 1, limit lower=-0.78539816339 upper=0.0 effort=5.0 velocity=1.0, mimic joint=zarm_l_finger_left_joint multiplier=-1 offset=0
- added joint zarm_r_finger_left_joint: type revolute, parent zarm_r7_end_effector, child zarm_r_finger_left, origin xyz=-0.02 0.035 0 rpy=0 0 0, axis 0 0 1, limit lower=0.0 upper=0.78539816339 effort=5.0 velocity=1.0
- added joint zarm_r_finger_right_joint: type revolute, parent zarm_r7_end_effector, child zarm_r_finger_right, origin xyz=-0.02 -0.035 0 rpy=0 0 0, axis 0 0 1, limit lower=-0.78539816339 upper=0.0 effort=5.0 velocity=1.0, mimic joint=zarm_r_finger_left_joint multiplier=-1 offset=0
- joint zarm_l6_joint: origin xyz=0 0 -0.132050000125748 rpy=0 0 0 -> xyz=0 0 -0.12 rpy=0 0 0
- joint zarm_l7_end_effector_joint: origin xyz=0 -0.03 -0.17 rpy=0 0 0 -> xyz=0 0 0 rpy=0 1.57079632679 0
- joint zarm_l7_joint: origin xyz=0 0 -0.0589999999999999 rpy=0 0 0 -> xyz=0 0 -0.14 rpy=0 0 0
- joint zarm_r6_joint: origin xyz=0 0 -0.132050000240097 rpy=0 0 0 -> xyz=0 0 -0.12 rpy=0 0 0
- joint zarm_r7_end_effector_joint: origin xyz=0 0.03 -0.17 rpy=0 0 0 -> xyz=0 0 0 rpy=0 1.57079632679 0
- joint zarm_r7_joint: origin xyz=0 0 -0.0589999999999999 rpy=0 0 0 -> xyz=0 0 -0.14 rpy=0 0 0

File: isaac_lab_data_collection/install/my_robot_description/share/my_robot_description/urdf/biped_s40_primitives.urdf (robot description, URDF)
Before this commit: robot my_robot_description, 50 links, 49 joints
Links:
- link base_link: geometry visual box size=0.25 0.18 0.4
- link camera: geometry visual box size=0.06 0.04 0.04
- link camera_base: geometry collision cylinder length=0.15 radius=0.03; visual mesh filename=camera_base.STL scale=1 1 1
- link leg_l1_link: geometry visual cylinder length=0.12 radius=0.05
- link leg_l2_link: geometry visual box size=0.12 0.08 0.18
- link leg_l3_link: geometry visual cylinder length=0.24 radius=0.045
- link leg_l4_link: geometry visual box size=0.1 0.08 0.2
- link leg_l5_link: geometry visual box size=0.09 0.07 0.12
- link leg_l6_link: geometry visual box size=0.16 0.09 0.05
- link leg_r1_link: geometry visual cylinder length=0.12 radius=0.05
- link leg_r2_link: geometry visual box size=0.12 0.08 0.18
- link leg_r3_link: geometry visual cylinder length=0.24 radius=0.045
- link leg_r4_link: geometry visual box size=0.1 0.08 0.2
- link leg_r5_link: geometry visual box size=0.09 0.07 0.12
- link leg_r6_link: geometry visual box size=0.16 0.09 0.05
- link zarm_l1_link: geometry visual cylinder length=0.12 radius=0.04
- link zarm_l2_link: geometry visual box size=0.1 0.08 0.14
- link zarm_l3_link: geometry visual cylinder length=0.26 radius=0.04
- link zarm_l4_link: geometry visual box size=0.08 0.08 0.18
- link zarm_l5_link: geometry visual box size=0.06 0.08 0.16
- link zarm_l6_link: geometry visual cylinder length=0.14 radius=0.03
- link zarm_l7_link: geometry visual box size=0.05 0.07 0.14
- link zarm_r1_link: geometry visual cylinder length=0.12 radius=0.04
- link zarm_r2_link: geometry visual box size=0.1 0.08 0.14
- link zarm_r3_link: geometry visual cylinder length=0.26 radius=0.04
- link zarm_r4_link: geometry visual box size=0.08 0.08 0.18
- link zarm_r5_link: geometry visual box size=0.06 0.08 0.16
- link zarm_r6_link: geometry visual cylinder length=0.14 radius=0.03
- link zarm_r7_link: geometry visual box size=0.05 0.07 0.14
- link zhead_1_link: geometry visual cylinder length=0.1 radius=0.05
- link zhead_2_link: geometry visual box size=0.16 0.14 0.2
